Commit message: New lizi world (wall patrol)

File: lizi_description/models/lizi.xacro (robot description, xacro)
@@ -75,5 +75,5 @@
         <pose>0.00740029995582005 -2.28205996951805E-05 -0.0185383676881744 0 0 0</pose>
         <inertial>
-          <pose>0 0 0 0 0 0</pose>
+          <pose>0 0 0.1 0 0 0</pose>
           <mass>0.737826</mass>
           <inertia>
@@ -87,5 +87,5 @@
         </inertial>
         <collision name='base_link_collision'>
-          <pose>0 0 0 0 -0 0</pose>
+          <pose>0 0 0 0 0 0</pose>
           <geometry>
             <mesh>

File: lizi_description/models/lizi_single_wall.xacro (robot description, xacro)
@@ -1,10 +1,9 @@
-<?xml version="1.0" ?>
-<!-- =================================================================================== -->
-<!-- |    This document was autogenerated by xacro from /home/blackpc/open-source-workspaces/models/src/lizi_description/models/lizi_single_wall.xacro | -->
-<!-- |    EDITING THIS FILE BY HAND IS NOT RECOMMENDED                                 | -->
-<!-- =================================================================================== -->
-<sdf version="1.4" xmlns:controller="http://playerstage.sourceforge.net/gazebo/xmlschema/#controller" xmlns:interface="http://playerstage.sourceforge.net/gazebo/xmlschema/#interface" xmlns:sensor="http://playerstage.sourceforge.net/gazebo/xmlschema/#sensor" xmlns:xacro="http://playerstage.sourceforge.net/gazebo/xmlschema/#interface">
-  <world name="default">
-    <light name="sun" type="directional">
+<?xml version="1.0"?>
+<sdf version='1.4' xmlns:sensor="http://playerstage.sourceforge.net/gazebo/xmlschema/#sensor"
+    xmlns:controller="http://playerstage.sourceforge.net/gazebo/xmlschema/#controller"
+    xmlns:interface="http://playerstage.sourceforge.net/gazebo/xmlschema/#interface"
+    xmlns:xacro="http://playerstage.sourceforge.net/gazebo/xmlschema/#interface">
+  <world name='default'>
+    <light name='sun' type='directional'>
       <cast_shadows>1</cast_shadows>
       <pose>0 0 10 0 -0 0</pose>
@@ -19,8 +18,8 @@
       <direction>0.5 0.1 -0.9</direction>
     </light>
-    <model name="ground_plane">
+    <model name='ground_plane'>
       <static>1</static>
-      <link name="link">
-        <collision name="collision">
+      <link name='link'>
+        <collision name='collision'>
           <geometry>
             <plane>
@@ -61,5 +60,5 @@
       </link>
     </model>
-    <physics type="ode">
+    <physics type='ode'>
       <max_step_size>0.001</max_step_size>
       <real_time_factor>1</real_time_factor>
@@ -72,7 +71,7 @@
       <shadows>1</shadows>
     </scene>
-    <model name="lizi_urdf">
+    <model name='lizi_urdf'>
       <pose>0 0 1 0 -0 0</pose>
-      <link name="base_link">
+      <link name='base_link'>
         <pose>0.00740029995582005 -2.28205996951805E-05 -0.0185383676881744 0 0 0</pose>
         <inertial>
@@ -88,29 +87,29 @@
           </inertia>
         </inertial>
-        <collision name="base_link_collision">
+        <collision name='base_link_collision'>
           <pose>0 0 0 0 0 0</pose>
           <geometry>
             <mesh>
               <scale>1 1 1</scale>
-              <uri>/home/blackpc/open-source-workspaces/models/src/lizi_description/meshes/base_link.STL</uri>
-            </mesh>
-          </geometry>
-          <max_contacts>10</max_contacts>
-          <surface>
-            <bounce/>
-            <friction>
-              <ode/>
-            </friction>
-            <contact>
-              <ode/>
-            </contact>
-          </surface>
-        </collision>
-        <visual name="base_link_visual">
-          <pose>0 0 0 0 -0 0</pose>
-          <geometry>
-            <mesh>
-              <scale>1 1 1</scale>
-              <uri>/home/blackpc/open-source-workspaces/models/src/lizi_description/meshes/base_link.STL</uri>
+              <uri>$(find lizi_description)/meshes/base_link.STL</uri>
+            </mesh>
+          </geometry>
+          <max_contacts>10</max_contacts>
+          <surface>
+            <bounce/>
+            <friction>
+              <ode/>
+            </friction>
+            <contact>
+              <ode/>
+            </contact>
+          </surface>
+        </collision>
+        <visual name='base_link_visual'>
+          <pose>0 0 0 0 -0 0</pose>
+          <geometry>
+            <mesh>
+              <scale>1 1 1</scale>
+              <uri>$(find lizi_description)/meshes/base_link.STL</uri>
             </mesh>
           </geometry>
@@ -130,5 +129,5 @@
         <gravity>1</gravity>
       </link>
-      <link name="FL_wheel">
+      <link name='FL_wheel'>
         <pose>0.074003 0.1825 -0.04145 0 -0 0</pose>
         <inertial>
@@ -144,29 +143,29 @@
           </inertia>
         </inertial>
-        <collision name="FL_wheel_collision">
-          <pose>0 0 0 0 -0 0</pose>
-          <geometry>
-            <mesh>
-              <scale>1 1 1</scale>
-              <uri>/home/blackpc/open-source-workspaces/models/src/lizi_description/meshes/FL_wheel.STL</uri>
-            </mesh>
-          </geometry>
-          <max_contacts>10</max_contacts>
-          <surface>
-            <bounce/>
-            <friction>
-              <ode/>
-            </friction>
-            <contact>
-              <ode/>
-            </contact>
-          </surface>
-        </collision>
-        <visual name="FL_wheel_visual">
-          <pose>0 0 0 0 -0 0</pose>
-          <geometry>
-            <mesh>
-              <scale>1 1 1</scale>
-              <uri>/home/blackpc/open-source-workspaces/models/src/lizi_description/meshes/FL_wheel.STL</uri>
+        <collision name='FL_wheel_collision'>
+          <pose>0 0 0 0 -0 0</pose>
+          <geometry>
+            <mesh>
+              <scale>1 1 1</scale>
+              <uri>$(find lizi_description)/meshes/FL_wheel.STL</uri>
+            </mesh>
+          </geometry>
+          <max_contacts>10</max_contacts>
+          <surface>
+            <bounce/>
+            <friction>
+              <ode/>
+            </friction>
+            <contact>
+              <ode/>
+            </contact>
+          </surface>
+        </collision>
+        <visual name='FL_wheel_visual'>
+          <pose>0 0 0 0 -0 0</pose>
+          <geometry>
+            <mesh>
+              <scale>1 1 1</scale>
+              <uri>$(find lizi_description)/meshes/FL_wheel.STL</uri>
             </mesh>
           </geometry>
@@ -186,5 +185,5 @@
         <gravity>1</gravity>
       </link>
-      <joint name="FL_Joint" type="revolute">
+      <joint name='FL_Joint' type='revolute'>
         <child>FL_wheel</child>
         <parent>base_link</parent>
@@ -198,5 +197,5 @@
         </axis>
       </joint>
-      <link name="FR_Wheel">
+      <link name='FR_Wheel'>
         <pose>0.074003 -0.1825 -0.04145 -1.0694e-16 1.4202e-32 0</pose>
         <inertial>
@@ -212,29 +211,29 @@
           </inertia>
         </inertial>
-        <collision name="FR_Wheel_collision">
-          <pose>0 0 0 0 -0 0</pose>
-          <geometry>
-            <mesh>
-              <scale>1 1 1</scale>
-              <uri>/home/blackpc/open-source-workspaces/models/src/lizi_description/meshes/FR_Wheel.STL</uri>
-            </mesh>
-          </geometry>
-          <max_contacts>10</max_contacts>
-          <surface>
-            <bounce/>
-            <friction>
-              <ode/>
-            </friction>
-            <contact>
-              <ode/>
-            </contact>
-          </surface>
-        </collision>
-        <visual name="FR_Wheel_visual">
-          <pose>0 0 0 0 -0 0</pose>
-          <geometry>
-            <mesh>
-              <scale>1 1 1</scale>
-              <uri>/home/blackpc/open-source-workspaces/models/src/lizi_description/meshes/FR_Wheel.STL</uri>
+        <collision name='FR_Wheel_collision'>
+          <pose>0 0 0 0 -0 0</pose>
+          <geometry>
+            <mesh>
+              <scale>1 1 1</scale>
+              <uri>$(find lizi_description)/meshes/FR_Wheel.STL</uri>
+            </mesh>
+          </geometry>
+          <max_contacts>10</max_contacts>
+          <surface>
+            <bounce/>
+            <friction>
+              <ode/>
+            </friction>
+            <contact>
+              <ode/>
+            </contact>
+          </surface>
+        </collision>
+        <visual name='FR_Wheel_visual'>
+          <pose>0 0 0 0 -0 0</pose>
+          <geometry>
+            <mesh>
+              <scale>1 1 1</scale>
+              <uri>$(find lizi_description)/meshes/FR_Wheel.STL</uri>
             </mesh>
           </geometry>
@@ -254,5 +253,5 @@
         <gravity>1</gravity>
       </link>
-      <joint name="FR_Joint" type="revolute">
+      <joint name='FR_Joint' type='revolute'>
         <child>FR_Wheel</child>
         <parent>base_link</parent>
@@ -266,5 +265,5 @@
         </axis>
       </joint>
-      <link name="RL_Wheel">
+      <link name='RL_Wheel'>
         <pose>-0.126 0.1825 -0.04145 0 -0 0</pose>
         <inertial>
@@ -280,29 +279,29 @@
           </inertia>
         </inertial>
-        <collision name="RL_Wheel_collision">
-          <pose>0 0 0 0 -0 0</pose>
-          <geometry>
-            <mesh>
-              <scale>1 1 1</scale>
-              <uri>/home/blackpc/open-source-workspaces/models/src/lizi_description/meshes/RL_Wheel.STL</uri>
-            </mesh>
-          </geometry>
-          <max_contacts>10</max_contacts>
-          <surface>
-            <bounce/>
-            <friction>
-              <ode/>
-            </friction>
-            <contact>
-              <ode/>
-            </contact>
-          </surface>
-        </collision>
-        <visual name="RL_Wheel_visual">
-          <pose>0 0 0 0 -0 0</pose>
-          <geometry>
-            <mesh>
-              <scale>1 1 1</scale>
-              <uri>/home/blackpc/open-source-workspaces/models/src/lizi_description/meshes/RL_Wheel.STL</uri>
+        <collision name='RL_Wheel_collision'>
+          <pose>0 0 0 0 -0 0</pose>
+          <geometry>
+            <mesh>
+              <scale>1 1 1</scale>
+              <uri>$(find lizi_description)/meshes/RL_Wheel.STL</uri>
+            </mesh>
+          </geometry>
+          <max_contacts>10</max_contacts>
+          <surface>
+            <bounce/>
+            <friction>
+              <ode/>
+            </friction>
+            <contact>
+              <ode/>
+            </contact>
+          </surface>
+        </collision>
+        <visual name='RL_Wheel_visual'>
+          <pose>0 0 0 0 -0 0</pose>
+          <geometry>
+            <mesh>
+              <scale>1 1 1</scale>
+              <uri>$(find lizi_description)/meshes/RL_Wheel.STL</uri>
             </mesh>
           </geometry>
@@ -322,5 +321,5 @@
         <gravity>1</gravity>
       </link>
-      <joint name="RL_Joint" type="revolute">
+      <joint name='RL_Joint' type='revolute'>
         <child>RL_Wheel</child>
         <parent>base_link</parent>
@@ -334,5 +333,5 @@
         </axis>
       </joint>
-      <link name="RR_Wheel">
+      <link name='RR_Wheel'>
         <pose>-0.126 -0.1825 -0.04145 -1.0694e-16 1.4202e-32 0</pose>
         <inertial>
@@ -348,29 +347,29 @@
           </inertia>
         </inertial>
-        <collision name="RR_Wheel_collision">
-          <pose>0 0 0 0 -0 0</pose>
-          <geometry>
-            <mesh>
-              <scale>1 1 1</scale>
-              <uri>/home/blackpc/open-source-workspaces/models/src/lizi_description/meshes/RR_Wheel.STL</uri>
-            </mesh>
-          </geometry>
-          <max_contacts>10</max_contacts>
-          <surface>
-            <bounce/>
-            <friction>
-              <ode/>
-            </friction>
-            <contact>
-              <ode/>
-            </contact>
-          </surface>
-        </collision>
-        <visual name="RR_Wheel_visual">
-          <pose>0 0 0 0 -0 0</pose>
-          <geometry>
-            <mesh>
-              <scale>1 1 1</scale>
-              <uri>/home/blackpc/open-source-workspaces/models/src/lizi_description/meshes/RR_Wheel.STL</uri>
+        <collision name='RR_Wheel_collision'>
+          <pose>0 0 0 0 -0 0</pose>
+          <geometry>
+            <mesh>
+              <scale>1 1 1</scale>
+              <uri>$(find lizi_description)/meshes/RR_Wheel.STL</uri>
+            </mesh>
+          </geometry>
+          <max_contacts>10</max_contacts>
+          <surface>
+            <bounce/>
+            <friction>
+              <ode/>
+            </friction>
+            <contact>
+              <ode/>
+            </contact>
+          </surface>
+        </collision>
+        <visual name='RR_Wheel_visual'>
+          <pose>0 0 0 0 -0 0</pose>
+          <geometry>
+            <mesh>
+              <scale>1 1 1</scale>
+              <uri>$(find lizi_description)/meshes/RR_Wheel.STL</uri>
             </mesh>
           </geometry>
@@ -390,5 +389,5 @@
         <gravity>1</gravity>
       </link>
-      <joint name="RR_Joint" type="revolute">
+      <joint name='RR_Joint' type='revolute'>
         <child>RR_Wheel</child>
         <parent>base_link</parent>
@@ -403,5 +402,5 @@
       </joint>
       <static>0</static>
-      <link name="hokuyo::link">
+      <link name='hokuyo::link'>
         <inertial>
           <mass>0.1</mass>
@@ -415,12 +414,12 @@
           </inertia>
         </inertial>
-        <visual name="visual">
-          <geometry>
-            <mesh>
-              <uri>/home/blackpc/open-source-workspaces/models/src/lizi_description/meshes/hokuyo.dae</uri>
-            </mesh>
-          </geometry>
-        </visual>
-        <collision name="collision-base">
+        <visual name='visual'>
+          <geometry>
+            <mesh>
+              <uri>$(find lizi_description)/meshes/hokuyo.dae</uri>
+            </mesh>
+          </geometry>
+        </visual>
+        <collision name='collision-base'>
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